File: Eng_Thesis.kicad_pcb (KiCad board)
At the start: 2 copper layers, 11 parts, among them IC1 ISO6721RBDR, J3 ST_Llink, U1 STM32F030C8Tx, U2 SN6507DGQ, U3 ADE7953xCP, U4 LD3985G33R_TSOT23, U5 SN75176AD, U6 LF50_TO252, U7 LD3985G33R_TSOT23, U8 ISO1541

Commit message: v.0.1
Parts:
- added C1: 100n, Capacitor_SMD:C_0805_2012Metric_Pad1.18x1.45mm_HandSolder, F.Cu at (39.6, 34.3)
- added C10: 1u, Capacitor_SMD:C_0805_2012Metric_Pad1.18x1.45mm_HandSolder, F.Cu at (39.0, 24.9)
- added C11: 100n, Capacitor_SMD:C_0805_2012Metric_Pad1.18x1.45mm_HandSolder, F.Cu at (43.4, 25.4)
- added C12: 2.2u, Capacitor_SMD:CP_Elec_4x5.3, F.Cu at (54.6, 29.6)
- added C13: 10n, Capacitor_SMD:C_0805_2012Metric_Pad1.18x1.45mm_HandSolder, F.Cu at (34.3, 31.9)
- added C14: 4.7u, Capacitor_Tantalum_SMD:CP_EIA-3216-18_Kemet-A_Pad1.58x1.35mm_HandSolder, F.Cu at (70.6, 56.8)
- added C15: 1u, Capacitor_SMD:C_0805_2012Metric_Pad1.18x1.45mm_HandSolder, F.Cu at (39.9, 27.9)
- added C16: 4.7u, Capacitor_Tantalum_SMD:CP_EIA-3216-18_Kemet-A_Pad1.58x1.35mm_HandSolder, F.Cu at (70.6, 52.6)
- added C19: 1u, Capacitor_SMD:C_0805_2012Metric_Pad1.18x1.45mm_HandSolder, F.Cu at (73.2, 41.1)
- added C2: 100n, Capacitor_SMD:C_0805_2012Metric_Pad1.18x1.45mm_HandSolder, F.Cu at (38.1, 40.6)
- added C21: 10u, Capacitor_SMD:C_0805_2012Metric_Pad1.18x1.45mm_HandSolder, F.Cu at (73.2, 34.9)
- added C22: 10n, Capacitor_SMD:C_0805_2012Metric_Pad1.18x1.45mm_HandSolder, F.Cu at (63.1, 38.9)
- added C23: 0.1u, Capacitor_SMD:C_0805_2012Metric_Pad1.18x1.45mm_HandSolder, F.Cu at (73.2, 37.0)
- added C24: 1u, Capacitor_SMD:C_0805_2012Metric_Pad1.18x1.45mm_HandSolder, F.Cu at (63.1, 41.0)
- added C25: 4.7u, Capacitor_Tantalum_SMD:CP_EIA-3216-18_Kemet-A_Pad1.58x1.35mm_HandSolder, F.Cu at (61.0, 63.8)
- added C26: 33n, Capacitor_SMD:C_0805_2012Metric_Pad1.18x1.45mm_HandSolder, F.Cu at (61.3, 76.2)
- added C27: 0.1u, Capacitor_SMD:C_0805_2012Metric_Pad1.18x1.45mm_HandSolder, F.Cu at (61.6, 61.7)
- added C29: 0.1u, Capacitor_SMD:C_0805_2012Metric_Pad1.18x1.45mm_HandSolder, F.Cu at (47.0, 61.0)
- added C3: 100n, Capacitor_SMD:C_0805_2012Metric_Pad1.18x1.45mm_HandSolder, F.Cu at (48.9, 45.6)
- added C30: 33n, Capacitor_SMD:C_0805_2012Metric_Pad1.18x1.45mm_HandSolder, F.Cu at (15.6, 73.4)
- added C31: 33n, Capacitor_SMD:C_0805_2012Metric_Pad1.18x1.45mm_HandSolder, F.Cu at (28.8, 73.4)
- added C32: 33n, Capacitor_SMD:C_0805_2012Metric_Pad1.18x1.45mm_HandSolder, F.Cu at (39.4, 72.6)
- added C33: 33n, Capacitor_SMD:C_0805_2012Metric_Pad1.18x1.45mm_HandSolder, F.Cu at (52.3, 72.6)
- added C34: 0.1u, Capacitor_SMD:C_0805_2012Metric_Pad1.18x1.45mm_HandSolder, F.Cu at (73.2, 54.7)
- added C35: 0.1u, Capacitor_SMD:C_0805_2012Metric_Pad1.18x1.45mm_HandSolder, F.Cu at (49.0, 60.9)
- added C36: 33n, Capacitor_SMD:C_0805_2012Metric_Pad1.18x1.45mm_HandSolder, F.Cu at (15.6, 69.3)
- added C37: 33n, Capacitor_SMD:C_0805_2012Metric_Pad1.18x1.45mm_HandSolder, F.Cu at (28.8, 69.3)
- added C38: 33n, Capacitor_SMD:C_0805_2012Metric_Pad1.18x1.45mm_HandSolder, F.Cu at (39.4, 68.6)
- added C39: 33n, Capacitor_SMD:C_0805_2012Metric_Pad1.18x1.45mm_HandSolder, F.Cu at (52.3, 68.6)
- added C4: 100n, Capacitor_SMD:C_0805_2012Metric_Pad1.18x1.45mm_HandSolder, F.Cu at (41.7, 32.3)
- added C41: 33n, Capacitor_SMD:C_1210_3225Metric_Pad1.33x2.70mm_HandSolder, F.Cu at (74.0, 72.6)
- added C42: 0.1u, Capacitor_SMD:C_0805_2012Metric_Pad1.18x1.45mm_HandSolder, F.Cu at (45.2, 51.8)
- added C43: 0.1u, Capacitor_SMD:C_0805_2012Metric_Pad1.18x1.45mm_HandSolder, F.Cu at (69.3, 54.7)
- added C44: 0.1u, Capacitor_SMD:C_0805_2012Metric_Pad1.18x1.45mm_HandSolder, F.Cu at (49.3, 51.8)
- added C45: 20p, Capacitor_SMD:C_0805_2012Metric_Pad1.18x1.45mm_HandSolder, F.Cu at (62.4, 52.6)
- added C46: 20p, Capacitor_SMD:C_0805_2012Metric_Pad1.18x1.45mm_HandSolder, F.Cu at (58.5, 52.6)
- added C5: 4,7u, Capacitor_SMD:C_0805_2012Metric_Pad1.18x1.45mm_HandSolder, F.Cu at (37.8, 27.9)
- added C6: 10u, Capacitor_Tantalum_SMD:CP_EIA-3216-18_Kemet-A_Pad1.58x1.35mm_HandSolder, F.Cu at (66.2, 62.6)
- added C7: 0.1u, Capacitor_SMD:C_0805_2012Metric_Pad1.18x1.45mm_HandSolder, B.Cu at (27.9, 31.5)
- added C8: 0.1u, Capacitor_SMD:C_0805_2012Metric_Pad1.18x1.45mm_HandSolder, F.Cu at (66.2, 52.6)
- added C9: 100n, Capacitor_SMD:C_0805_2012Metric_Pad1.18x1.45mm_HandSolder, F.Cu at (31.0, 49.7)
- added D1: LED, LED_SMD:LED_0603_1608Metric_Pad1.05x0.95mm_HandSolder, F.Cu at (49.5, 33.0)
- added D2: LED, LED_SMD:LED_0603_1608Metric_Pad1.05x0.95mm_HandSolder, F.Cu at (46.7, 28.4)
- added D4: D_Zener, Diode_SMD:D_MELF, B.Cu at (37.0, 20.3)
- added D5: BAT165E6327HTSA1, Diode_SMD:D_SOD-323F, F.Cu at (69.0, 34.2)
- added D6: BAT165E6327HTSA1, Diode_SMD:D_SOD-323F, F.Cu at (64.5, 34.2)
- added D7: LED, LED_SMD:LED_0603_1608Metric_Pad1.05x0.95mm_HandSolder, F.Cu at (76.7, 40.1)
- added D8: LED, LED_SMD:LED_0603_1608Metric_Pad1.05x0.95mm_HandSolder, F.Cu at (63.0, 44.8)
- added F1: Fuse, Fuse:Fuse_2920_7451Metric_Pad2.10x5.45mm_HandSolder, F.Cu at (39.0, 17.8)
- added J2: Conn_01x03_Socket, Connector_PinSocket_2.54mm:PinSocket_1x03_P2.54mm_Vertical, F.Cu at (15.0, 48.1)
- added J5: Conn_01x02_Socket, LibLoader:TB508P2PBL, F.Cu at (19.6, 33.3)
- added J6: Jack-DC, LibLoader:PCGK21, F.Cu at (27.0, 25.1)
- added J7: Screw_Terminal_01x02, LibLoader:TB508P2PBL, F.Cu at (69.2, 82.2)
- added J8: Screw_Terminal_01x02, LibLoader:TB508P2PBL, F.Cu at (24.8, 82.4)
- added J9: Screw_Terminal_01x02, LibLoader:TB508P2PBL, F.Cu at (48.4, 82.2)
- added JP1: SolderJumper_2_Open, Jumper:SolderJumper-2_P1.3mm_Open_TrianglePad1.0x1.5mm, F.Cu at (34.8, 36.8)
- added Q1: Q_PMOS_GSD, Package_TO_SOT_SMD:SOT-23_Handsoldering, B.Cu at (38.1, 16.5)
- added R1: 4.7k, Resistor_SMD:R_0805_2012Metric_Pad1.20x1.40mm_HandSolder, B.Cu at (40.1, 52.3)
- added R10: 1k, Resistor_SMD:R_0805_2012Metric_Pad1.20x1.40mm_HandSolder, F.Cu at (45.5, 33.0)
- added R11: 1k, Resistor_SMD:R_0805_2012Metric_Pad1.20x1.40mm_HandSolder, F.Cu at (35.6, 22.9)
- added R12: 1k, Resistor_SMD:R_0805_2012Metric_Pad1.20x1.40mm_HandSolder, F.Cu at (50.8, 28.4)
- added R14: 21K, Resistor_SMD:R_0805_2012Metric_Pad1.20x1.40mm_HandSolder, F.Cu at (62.7, 15.1)
- added R16: 4.7k, Resistor_SMD:R_0805_2012Metric_Pad1.20x1.40mm_HandSolder, F.Cu at (55.2, 39.1)
- added R17: 4.7k, Resistor_SMD:R_0805_2012Metric_Pad1.20x1.40mm_HandSolder, F.Cu at (55.2, 35.0)
- added R18: 50K, Resistor_SMD:R_0805_2012Metric_Pad1.20x1.40mm_HandSolder, F.Cu at (62.7, 17.0)
- added R2: 10k, Resistor_SMD:R_0805_2012Metric_Pad1.20x1.40mm_HandSolder, B.Cu at (32.5, 31.0)
- added R20: 1k, Resistor_SMD:R_0805_2012Metric_Pad1.20x1.40mm_HandSolder, F.Cu at (73.2, 39.0)
- added R21: 1k, Resistor_SMD:R_0805_2012Metric_Pad1.20x1.40mm_HandSolder, F.Cu at (63.1, 43.0)
- added R22: 1k, Resistor_SMD:R_0805_2012Metric_Pad1.20x1.40mm_HandSolder, F.Cu at (63.5, 76.2)
- added R23: 110k, Resistor_SMD:R_0805_2012Metric_Pad1.20x1.40mm_HandSolder, F.Cu at (65.8, 76.2)
- added R24: 30m, Resistor_SMD:R_2512_6332Metric_Pad1.40x3.35mm_HandSolder, F.Cu at (19.7, 74.2)
- added R25: 30m, Resistor_SMD:R_2512_6332Metric_Pad1.40x3.35mm_HandSolder, F.Cu at (24.8, 74.0)
- added R26: 30m, Resistor_SMD:R_2512_6332Metric_Pad1.40x3.35mm_HandSolder, F.Cu at (43.3, 73.7)
- added R27: 30m, Resistor_SMD:R_2512_6332Metric_Pad1.40x3.35mm_HandSolder, F.Cu at (48.4, 73.7)
- added R28: 100, Resistor_SMD:R_0805_2012Metric_Pad1.20x1.40mm_HandSolder, F.Cu at (16.6, 76.3)
- added R29: 100, Resistor_SMD:R_0805_2012Metric_Pad1.20x1.40mm_HandSolder, F.Cu at (27.9, 76.3)
- added R3: 4.7k, Resistor_SMD:R_0805_2012Metric_Pad1.20x1.40mm_HandSolder, F.Cu at (44.1, 48.9)
- added R30: 100, Resistor_SMD:R_0805_2012Metric_Pad1.20x1.40mm_HandSolder, F.Cu at (40.3, 75.8)
- added R31: 100, Resistor_SMD:R_0805_2012Metric_Pad1.20x1.40mm_HandSolder, F.Cu at (51.4, 75.8)
- added R32: 200k, Resistor_SMD:R_0805_2012Metric_Pad1.20x1.40mm_HandSolder, F.Cu at (68.0, 76.2)
- added R33: 200k, Resistor_SMD:R_0805_2012Metric_Pad1.20x1.40mm_HandSolder, F.Cu at (70.2, 76.2)
- added R34: 1k, Resistor_SMD:R_0805_2012Metric_Pad1.20x1.40mm_HandSolder, F.Cu at (15.6, 71.4)
- added R35: 1k, Resistor_SMD:R_0805_2012Metric_Pad1.20x1.40mm_HandSolder, F.Cu at (28.8, 71.4)
- added R36: 1k, Resistor_SMD:R_0805_2012Metric_Pad1.20x1.40mm_HandSolder, F.Cu at (39.4, 70.6)
- added R37: 1k, Resistor_SMD:R_0805_2012Metric_Pad1.20x1.40mm_HandSolder, F.Cu at (52.3, 70.6)
- added R38: 1k, Resistor_SMD:R_0805_2012Metric_Pad1.20x1.40mm_HandSolder, F.Cu at (72.5, 76.2)
- added R39: 4.7k, Resistor_SMD:R_0805_2012Metric_Pad1.20x1.40mm_HandSolder, F.Cu at (55.1, 63.0)
- added R4: 10k, Resistor_SMD:R_0805_2012Metric_Pad1.20x1.40mm_HandSolder, F.Cu at (27.9, 29.5)
- added R40: 4.7k, Resistor_SMD:R_0805_2012Metric_Pad1.20x1.40mm_HandSolder, F.Cu at (58.8, 59.2)
- added R41: 4.7k, Resistor_SMD:R_0805_2012Metric_Pad1.20x1.40mm_HandSolder, F.Cu at (58.5, 55.4)
- added R42: 4.7k, Resistor_SMD:R_0805_2012Metric_Pad1.20x1.40mm_HandSolder, F.Cu at (52.3, 62.9)
- added R43: 4.7k, Resistor_SMD:R_0805_2012Metric_Pad1.20x1.40mm_HandSolder, F.Cu at (42.7, 62.6)
- added R44: 4.7k, Resistor_SMD:R_0805_2012Metric_Pad1.20x1.40mm_HandSolder, F.Cu at (44.7, 62.6)
- added R5: 4.7k, Resistor_SMD:R_0805_2012Metric_Pad1.20x1.40mm_HandSolder, F.Cu at (53.2, 46.6)
- added R6: 4.7k, Resistor_SMD:R_0805_2012Metric_Pad1.20x1.40mm_HandSolder, F.Cu at (54.4, 50.8)
- added R8: 10k, Resistor_SMD:R_0805_2012Metric_Pad1.20x1.40mm_HandSolder, B.Cu at (43.2, 37.1)
- added R9: 10k, Resistor_SMD:R_0805_2012Metric_Pad1.20x1.40mm_HandSolder, F.Cu at (34.9, 39.8)
- added SW1: MODBUS_ADDR, LibLoader:SDA08H1BD, F.Cu at (17.1, 61.0)
- added SW2: RESET, LibLoader:TL3305BF160QG, F.Cu at (37.6, 48.3)
- added T2: 78250MC-R, LibLoader:SOP254P1270X660-6N, F.Cu at (67.7, 25.9)
- added TP3: TestPoint, TestPoint:TestPoint_Pad_1.5x1.5mm, F.Cu at (53.8, 24.9)
- added TP6: 3V3_ISO, TestPoint:TestPoint_Pad_1.5x1.5mm, F.Cu at (67.2, 43.9)
- added Y2: 3.58 MHz, Crystal:Crystal_SMD_HC49-SD_HandSoldering, F.Cu at (66.8, 48.9)
- U1: renamed from U5; moved to B.Cu
- moved U4 94.7 mm to (35.1, 27.8), turned to -90 degrees
- moved U1 87.9 mm to (29.2, 35.6), turned to 180 degrees
- moved J1 87.0 mm to (17.3, 44.2), turned to 90 degrees
- moved U3 86.8 mm to (49.0, 19.9), turned to 90 degrees
- moved U5 78.2 mm to (67.8, 16.3), turned to 180 degrees
- moved U2 70.4 mm to (44.5, 39.4)
- moved U8 68.3 mm to (43.2, 56.9), turned to -90 degrees
- moved L1 67.9 mm to (68.0, 37.4)
- moved U6 61.4 mm to (68.0, 41.0), turned to 180 degrees
- moved U7 57.3 mm to (63.8, 57.0), turned to 90 degrees
- moved IC1 56.9 mm to (52.8, 56.9), turned to 90 degrees
- renumbered J3 to J1, U1 to U2, U6 to U3, U2 to U5, U7 to U6, U3 to U7
Connections:
- IC1 pad 6: /Measurement_Circuit/STM_ADE_RST -> /STM_ADE_IRQ
- IC1 pad 7: /Measurement_Circuit/STM_ADE_IRQ -> /STM_ADE_RST
- IC1 pad 8: +3V3 -> +3.3V
- U2 pad 1: +3V3 -> +3.3V
- U2 pad 18: Net-(U1-PB0) -> unconnected-(U2-PB0-Pad18)
- U2 pad 19: Net-(U1-PB1) -> unconnected-(U2-PB1-Pad19)
- U2 pad 20: Net-(U1-PB2) -> unconnected-(U2-PB2-Pad20)
- U2 pad 21: /I2C2_SCL -> /I2C_SCL
- U2 pad 22: /I2C2_SDA -> /I2C_SDA
- U2 pad 24: +3V3 -> +3.3V
- U2 pad 25: unconnected-(U1-PB12-Pad25) -> /MB_ADDR_8
- U2 pad 26: unconnected-(U1-PB13-Pad26) -> /MB_ADDR_7
- U2 pad 27: unconnected-(U1-PB14-Pad27) -> /MB_ADDR_6
- U2 pad 28: unconnected-(U1-PB15-Pad28) -> /MB_ADDR_5
- U2 pad 29: unconnected-(U1-PA8-Pad29) -> /MB_ADDR_4
- U2 pad 32: unconnected-(U1-PA11-Pad32) -> /MB_ADDR_3
- U2 pad 35: unconnected-(U1-PF6-Pad35) -> /MB_ADDR_2
- U2 pad 36: unconnected-(U1-PF7-Pad36) -> /MB_ADDR_1
- U2 pad 39: Net-(U1-PB3) -> unconnected-(U2-PB3-Pad39)
- U2 pad 40: Net-(U1-PB4) -> unconnected-(U2-PB4-Pad40)
- U2 pad 41: Net-(U1-PB5) -> unconnected-(U2-PB5-Pad41)
- U2 pad 42: Net-(U1-PB6) -> unconnected-(U2-PB6-Pad42)
- U2 pad 43: Net-(U1-PB7) -> unconnected-(U2-PB7-Pad43)
- U2 pad 48: +3V3 -> +3.3V
- U2 pad 5: /HSE_IN -> unconnected-(U2-PF0-Pad5)
- U2 pad 6: /HSE_OUT -> unconnected-(U2-PF1-Pad6)
- U2 pad 9: +3V3 -> +3.3V
- U5 pad 11: (no net) -> GND
- U7 pad 16: GNDA -> GND_ISO
- U7 pad 7: +3V3 -> +3V3_ISO
- U7 pad 8: +3V3 -> +3V3_ISO
- U8 pad 1: +3V3 -> +3.3V
- U8 pad 2: /Measurement_Circuit/I2C2_SCL -> /I2C_SDA
- U8 pad 3: /Measurement_Circuit/I2C2_SDA -> /I2C_SCL
Routing:
- net /Measurement_Circuit/IAP: track 0.00 -> 59.7 mm
- net GND_ISO: track 0.00 -> 58.5 mm, vias 0 -> 66
- net /STM_ADE_IRQ: track 0.00 -> 48.5 mm, vias 0 -> 2
- net /Measurement_Circuit/IAN: track 0.00 -> 47.0 mm
- net /Measurement_Circuit/IBP: track 0.00 -> 45.6 mm
- net GND: track 0.00 -> 43.9 mm, vias 0 -> 105
- net Net-(U5-EN/UVLO): track 0.00 -> 39.8 mm
- net +3.3V: track 0.00 -> 39.6 mm, vias 0 -> 19
- net /MB_ADDR_1: track 0.00 -> 39.5 mm, vias 0 -> 1
- net /MB_ADDR_2: track 0.00 -> 36.1 mm, vias 0 -> 1
- net /SWDIO: track 0.00 -> 34.3 mm, vias 0 -> 1
- net /SWCLK: track 0.00 -> 34.2 mm, vias 0 -> 1
- net /RS485_RX: track 0.00 -> 33.9 mm, vias 0 -> 1
- net /Measurement_Circuit/IBN: track 0.00 -> 33.8 mm
- net /MB_ADDR_3: track 0.00 -> 33.0 mm, vias 0 -> 1
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- added copper zone on F.Cu, net +3.3V
- added copper zone on In2.Cu, net +3.3V
- added copper zone on In2.Cu, net +3V3_ISO
- added copper zone on In2.Cu, net +5V
- added copper zone on B.Cu, net GND
- added copper zone on F.Cu, net GND
- added copper zone on In1.Cu, net GND
- added copper zone on B.Cu, net GND_ISO
- added copper zone on F.Cu, net GND_ISO
- added copper zone on In1.Cu, net GND_ISO
- added copper zone on F.Cu, net Net-(D5-K)
- added copper zone on B.Cu, net Net-(Q1-D)
- added copper zone on In2.Cu, net VCC
Other:
- board outline added: 65.5 x 74.8 mm
- copper layers 2 -> 4
- board text added: "230VAC"
- board text added: "3V3-SWCLK-GND-SWDIO-NRST-SWO"
- board text added: "A"
- board text added: "B"
- board text added: "Modbus address"
- board text added: "Neutral current IB"
- board text added: "Phase current IA"
- board text added: "RS485"
- board text added: "RS_DE"
- board text added: "Reset"
- board text added: "TX-RX-GND"
- board text added: "UART"
- board text added: "Voltage"
