File: Eng_Thesis.kicad_sch (KiCad schematic)
At the start: 33 parts, among them J1 ST_Llink, J2 Conn_02x07_Counter_Clockwise, J3 Conn_02x07_Counter_Clockwise, J4 Conn_02x07_Counter_Clockwise, J5 Conn_01x02_Socket, SW1 MODBUS_ADDR, SW2 RESET, U1 SN75176AD, U2 STM32F030C8Tx, Y1 38MHz

Commit message: v.0.1
Parts:
- removed C6, C8: 20p, Capacitor_SMD:C_0805_2012Metric_Pad1.18x1.45mm_HandSolder, symbol Device:C
- removed J2, J3, J4: Conn_02x07_Counter_Clockwise, Connector_PinHeader_2.54mm:PinHeader_2x07_P2.54mm_Vertical, symbol Connector_Generic:Conn_02x07_Counter_Clockwise
- removed R7: 390R, Resistor_SMD:R_0805_2012Metric_Pad1.20x1.40mm_HandSolder, symbol Device:R
- removed TP1, TP2: TestPoint, TestPoint:TestPoint_Pad_1.5x1.5mm, symbol Connector:TestPoint
- removed Y1: 38MHz, Crystal:Crystal_SMD_HC49-SD_HandSoldering, symbol Device:Crystal
- added J2: Conn_01x03_Socket, Connector_PinSocket_2.54mm:PinSocket_1x03_P2.54mm_Vertical, symbol Connector:Conn_01x03_Socket
Connections:
- net +3V3 is gone; now on net +3.3V: R1.1, R3.1, R5.1, R6.1, R8.1, R9.1, U2.1 (VDD), U2.24 (VDD), U2.48 (VDD), U2.9 (VDDA)
- net GND: now also J2.3 (Pin_3)
- net UART_TRACE_RX: now also J2.2 (Pin_2)
- net UART_TRACE_TX: now also J2.1 (Pin_1)
- net HSE_IN: no longer names the net of U2.5 (PF0)
- net HSE_OUT: no longer names the net of U2.6 (PF1)
- net I2C2_SCL renamed I2C_SCL
- net I2C2_SDA renamed I2C_SDA
- net PA4: no longer names the net of U2.14 (PA4)
- net PA5: no longer names the net of U2.15 (PA5)
- net PA6: no longer names the net of U2.16 (PA6)
- net PA7: no longer names the net of U2.17 (PA7)
- net PB0: no longer names the net of U2.18 (PB0)
- net PB1: no longer names the net of U2.19 (PB1)
- net PB2: no longer names the net of U2.20 (PB2)
- net PB8_Golpin2: no longer names the net of U2.45 (PB8)
- net PB9_Golpin2: no longer names the net of U2.46 (PB9)
- no-connect marks 0 -> 20
Other:
- sheet Measurement_Circuit ports: added I2C_SCL, I2C_SDA, STM_ADE_IRQ, STM_ADE_RST; removed none
- moved on the sheet: J1
