File: Power.kicad_sch (KiCad schematic)
At the start: 45 parts, among them J6 Screw_Terminal_01x03, T1 230/6, T2 78250MC-R, U3 LF50_TO252, U4 LD3985G33R_TSOT23, U5 SN6507DGQ, U6 LD3985G33R_TSOT23

Commit message: v.0.1
Parts:
- removed C14: 100n, Capacitor_THT:C_Rect_L18.0mm_W6.0mm_P15.00mm_FKS3_FKP3, symbol Device:C
- removed C16, C17: 2,2n, Capacitor_THT:C_Disc_D10.5mm_W5.0mm_P7.50mm, symbol Device:C
- removed C18: 100u, Capacitor_SMD:C_0805_2012Metric_Pad1.18x1.45mm_HandSolder, symbol Device:C
- removed C20: 6800u, Capacitor_THT:CP_Radial_D18.0mm_P7.50mm, symbol Device:C_Polarized
- removed D3: LED, LED_SMD:LED_0603_1608Metric_Pad1.05x0.95mm_HandSolder, symbol Device:LED
- removed D4: ABS8, Diode_SMD:Diode_Bridge_Diotec_ABS, symbol Diode_Bridge:ABS8
- removed J6: Screw_Terminal_01x03, LibLoader:XY126V-3P, symbol Connector:Screw_Terminal_01x03
- removed R13: 1k, Resistor_SMD:R_0805_2012Metric_Pad1.20x1.40mm_HandSolder, symbol Device:R
- removed R19: 100R, Resistor_SMD:R_2512_6332Metric_Pad1.40x3.35mm_HandSolder, symbol Device:R
- removed T1: 230/6, Transformer_THT:TSZZ4.5003M, symbol Device:Transformer_1P_1S
- removed TP4: 3V3, TestPoint:TestPoint_Pad_1.5x1.5mm, symbol Connector:TestPoint
- removed TP5: BrOut, TestPoint:TestPoint_Pad_1.5x1.5mm, symbol Connector:TestPoint
- added D4: D_Zener, Diode_SMD:D_MELF, symbol Device:D_Zener
- added J6: Jack-DC, LibLoader:PCGK21, symbol Connector:Jack-DC
- added Q1: Q_PMOS_GSD, Package_TO_SOT_SMD:SOT-23_Handsoldering, symbol Device:Q_PMOS_GSD
- F1: value 315mA -> Fuse
- R11: value 1M -> 1k; footprint Resistor_SMD:R_1206_3216Metric_Pad1.30x1.75mm_HandSolder -> Resistor_SMD:R_0805_2012Metric_Pad1.20x1.40mm_HandSolder
Connections:
- net GND: now also R11.2, J6.2
- net VCC: now also D4.1 (K), Q1.2 (S)
- net at R11.1: now also D4.2 (A), Q1.1 (G); no longer F1.2
- net at F1.1: now also J6.1
- new net: F1.2, Q1.3 (D)
